File: Electronics/KiCad/enigma_encoder/enigma_encoder.kicad_pcb (KiCad board)
At the start: 4 copper layers, 266.2 x 144.3 mm, 59 parts, among them IC1 EPM570T144C5N, J1 53258-0329, J10 53258-0329, J11 53258-0329, J12 53258-0329, J13 53258-0329, J14 53258-0329, J15 53258-0329, J16 53258-0329, J17 53258-0329, J18 53258-0329, J19 53258-0329, J2 53258-0329, J20 53258-0329, J21 53258-0329, J22 53258-0329, J23 53258-0329, J24 53258-0329, J25 53258-0329, J26 53258-0329, J27 53258-0329, J28 53258-0329, J29 53258-0329, J3 53258-0329, J30 53258-0329, J31 53258-0329, J32 53258-0329, J33 53258-0329, J34 53258-0329, J35 53258-0329, J36 53258-0329, J37 Conn_02x06_Odd_Even, J38 Conn_02x05_Odd_Even, J4 53258-0329, J5 53258-0329, J6 53258-0329, J7 53258-0329, J8 53258-0329, J9 53258-0329, Y1 SIT8918BAU71-33E-50.000000G

Commit message: KiCAD Encoder: Move decoupling caps and traces.
Parts:
- removed J10, J11, J12, J13, J14, J15, J16, J17, J18, J19, J20, J21, J22, J23, J24, J25, J26, J27, J28, J29, J30, J31, J32, J33, J34, J35, J36, J5, J6, J7, J8, J9: 53258-0329, SamacSys_Footprints:SHDR3W120P0X350_1X3_1260X760X1050P
- removed J37: Conn_02x06_Odd_Even, Connector_IDC:IDC-Header_2x06_P2.54mm_Vertical
- removed J38: Conn_02x05_Odd_Even, Connector_IDC:IDC-Header_2x05_P2.54mm_Vertical
- C1, C2, C3, C7, C8, C9: moved to F.Cu
- J1, J2: value 53258-0329 -> Conn_02x20_Odd_Even; footprint SamacSys_Footprints:SHDR3W120P0X350_1X3_1260X760X1050P -> Connector_IDC:IDC-Header_2x20_P2.54mm_Vertical
- J3: value 53258-0329 -> Conn_02x06_Odd_Even; footprint SamacSys_Footprints:SHDR3W120P0X350_1X3_1260X760X1050P -> Connector_IDC:IDC-Header_2x06_P2.54mm_Vertical
- J4: value 53258-0329 -> Conn_02x05_Odd_Even; footprint SamacSys_Footprints:SHDR3W120P0X350_1X3_1260X760X1050P -> Connector_IDC:IDC-Header_2x05_P2.54mm_Vertical
- moved J2 175.0 mm to (190.0, 82.0), turned to 180 degrees
- moved J3 164.8 mm to (181.9, 19.5), turned to -90 degrees
- moved J4 120.6 mm to (131.5, 19.4), turned to -90 degrees
- moved J1 99.6 mm to (119.7, 33.5), turned to 0 degrees
- moved C8 1.75 mm to (164.4, 42.0)
- moved C7 1.71 mm to (164.4, 47.7)
- moved C9 1.71 mm to (164.4, 37.7)
- moved C2 1.68 mm to (139.6, 42.5)
- moved C1 1.67 mm to (139.6, 38.2)
- moved C3 1.64 mm to (139.6, 47.2)
- moved C5 0.25 mm to (152.2, 54.7)
- moved C11 0.24 mm to (152.2, 29.7)
Connections:
- J1 pad 3: /KEY_IN_01 -> /KEY_IN_02
- J2 pad 1: /KEY_IN_02 -> /KEY_IN_19
- J2 pad 2: /KEY_OUT_02 -> /KEY_OUT_19
- J2 pad 3: /KEY_IN_02 -> /KEY_IN_20
- J3 pad 1: /KEY_IN_03 -> /BIN_IN_01
- J3 pad 2: /KEY_OUT_03 -> /BIN_OUT_01
- J3 pad 3: /KEY_IN_03 -> /BIN_IN_02
- J4 pad 1: /KEY_IN_04 -> /JTAG_TCK
- J4 pad 2: /KEY_OUT_04 -> GND
- J4 pad 3: /KEY_IN_04 -> /JTAG_TDO
Routing:
- net /KEY_OUT_10: track 162.9 -> 23.8 mm
- net /KEY_IN_10: track 161.7 -> 26.5 mm
- net /KEY_OUT_09: track 157.5 -> 23.1 mm
- net /KEY_IN_11: track 158.8 -> 27.2 mm
- net /KEY_IN_09: track 156.3 -> 25.9 mm
- net /KEY_OUT_11: track 153.6 -> 24.6 mm
- net /KEY_OUT_08: track 152.5 -> 25.3 mm, vias 0 -> 2
- net /KEY_IN_08: track 151.4 -> 25.6 mm
- net /KEY_OUT_07: track 147.3 -> 22.3 mm
- net /KEY_OUT_27: track 153.7 -> 31.9 mm
- net /KEY_IN_07: track 146.1 -> 25.0 mm
- net /KEY_OUT_06: track 142.0 -> 21.7 mm
- net /KEY_OUT_12: track 144.6 -> 24.7 mm
- net /KEY_IN_27: track 154.9 -> 35.2 mm
- net /KEY_IN_12: track 147.0 -> 28.9 mm
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- removed copper zone on B.Cu, net /KEY_IN_01
- removed copper zone on B.Cu, net /KEY_IN_02
- removed copper zone on B.Cu, net /KEY_IN_03
- removed copper zone on B.Cu, net /KEY_IN_04
- removed copper zone on B.Cu, net /KEY_IN_05
- removed copper zone on B.Cu, net /KEY_IN_06
- removed copper zone on B.Cu, net /KEY_IN_07
- removed copper zone on B.Cu, net /KEY_IN_08
- removed copper zone on B.Cu, net /KEY_IN_09
- removed copper zone on B.Cu, net /KEY_IN_10
- removed copper zone on B.Cu, net /KEY_IN_11
- removed copper zone on B.Cu, net /KEY_IN_12
- removed copper zone on B.Cu, net /KEY_IN_13
- removed copper zone on B.Cu, net /KEY_IN_14
- removed copper zone on B.Cu, net /KEY_IN_15
- removed copper zone on B.Cu, net /KEY_IN_16
- removed copper zone on B.Cu, net /KEY_IN_17
- removed copper zone on B.Cu, net /KEY_IN_18
- removed copper zone on B.Cu, net /KEY_IN_19
- removed copper zone on B.Cu, net /KEY_IN_20
- removed copper zone on B.Cu, net /KEY_IN_21
- removed copper zone on B.Cu, net /KEY_IN_22
- removed copper zone on B.Cu, net /KEY_IN_23
- removed copper zone on B.Cu, net /KEY_IN_24
- removed copper zone on B.Cu, net /KEY_IN_25
- removed copper zone on B.Cu, net /KEY_IN_26
- removed copper zone on B.Cu, net /KEY_IN_27
- removed copper zone on B.Cu, net /KEY_IN_28
- removed copper zone on B.Cu, net /KEY_IN_29
- removed copper zone on B.Cu, net /KEY_IN_30
- removed copper zone on B.Cu, net /KEY_IN_31
- removed copper zone on B.Cu, net /KEY_IN_32
- removed copper zone on B.Cu, net /KEY_IN_33
- removed copper zone on B.Cu, net /KEY_IN_34
- removed copper zone on B.Cu, net /KEY_IN_35
- removed copper zone on B.Cu, net /KEY_IN_36
Other:
- board size 266.2 x 144.3 mm -> 81.4 x 76 mm
- board text added: "C6"
