File: Electronics/KiCad/enigma_encoder/enigma_encoder.kicad_sch (KiCad schematic)
At the start: 59 parts, among them IC1 EPM570T144C5N, J1 53258-0329, J10 53258-0329, J11 53258-0329, J12 53258-0329, J13 53258-0329, J14 53258-0329, J15 53258-0329, J16 53258-0329, J17 53258-0329, J18 53258-0329, J19 53258-0329, J2 53258-0329, J20 53258-0329, J21 53258-0329, J22 53258-0329, J23 53258-0329, J24 53258-0329, J25 53258-0329, J26 53258-0329, J27 53258-0329, J28 53258-0329, J29 53258-0329, J3 53258-0329, J30 53258-0329, J31 53258-0329, J32 53258-0329, J33 53258-0329, J34 53258-0329, J35 53258-0329, J36 53258-0329, J37 Conn_02x06_Odd_Even, J38 Conn_02x05_Odd_Even, J4 53258-0329, J5 53258-0329, J6 53258-0329, J7 53258-0329, J8 53258-0329, J9 53258-0329, Y1 SIT8918BAU71-33E-50.000000G

Commit message: KiCAD Encoder: Move decoupling caps and traces.
Parts:
- removed J1, J10, J11, J12, J13, J14, J15, J16, J17, J18, J19, J2, J20, J21, J22, J23, J24, J25, J26, J27, J28, J29, J3, J30, J31, J32, J33, J34, J35, J36, J4, J5, J6, J7, J8, J9: 53258-0329, SamacSys_Footprints:SHDR3W120P0X350_1X3_1260X760X1050P, symbol SamacSys_Parts:53258-0329
- removed J37: Conn_02x06_Odd_Even, Connector_IDC:IDC-Header_2x06_P2.54mm_Vertical, symbol Connector_Generic:Conn_02x06_Odd_Even
- removed J38: Conn_02x05_Odd_Even, Connector_IDC:IDC-Header_2x05_P2.54mm_Vertical, symbol Connector_Generic:Conn_02x05_Odd_Even
- added J1, J2: Conn_02x20_Odd_Even, Connector_IDC:IDC-Header_2x20_P2.54mm_Vertical, symbol Connector_Generic:Conn_02x20_Odd_Even
- added J3: Conn_02x06_Odd_Even, Connector_IDC:IDC-Header_2x06_P2.54mm_Vertical, symbol Connector_Generic:Conn_02x06_Odd_Even
- added J4: Conn_02x05_Odd_Even, Connector_IDC:IDC-Header_2x05_P2.54mm_Vertical, symbol Connector_Generic:Conn_02x05_Odd_Even
Connections:
- net BIN_IN_01: now also J3.1 (Pin_1)
- net BIN_IN_02: now also J3.3 (Pin_3)
- net BIN_IN_03: now also J3.5 (Pin_5)
- net BIN_IN_04: now also J3.7 (Pin_7)
- net BIN_IN_05: now also J3.9 (Pin_9)
- net BIN_IN_06: now also J3.11 (Pin_11)
- net BIN_OUT_01: now also J3.2 (Pin_2)
- net BIN_OUT_02: now also J3.4 (Pin_4)
- net BIN_OUT_03: now also J3.6 (Pin_6)
- net BIN_OUT_04: now also J3.8 (Pin_8)
- net BIN_OUT_05: now also J3.10 (Pin_10)
- net BIN_OUT_06: now also J3.12 (Pin_12)
- net GND: now also J4.10 (Pin_10), J4.2 (Pin_2)
- net JTAG_TCK: now also J4.1 (Pin_1)
- net JTAG_TDI: now also J4.9 (Pin_9)
- net JTAG_TDO: now also J4.3 (Pin_3)
- net JTAG_TMS: now also J4.5 (Pin_5)
- net KEY_IN_01: now also J1.1 (Pin_1)
- net KEY_IN_02: now also J1.3 (Pin_3)
- net KEY_IN_03: now also J1.5 (Pin_5)
- net KEY_IN_04: now also J1.7 (Pin_7)
- net KEY_IN_05: now also J1.9 (Pin_9)
- net KEY_IN_06: now also J1.11 (Pin_11)
- net KEY_IN_07: now also J1.13 (Pin_13)
- net KEY_IN_08: now also J1.15 (Pin_15)
- net KEY_IN_09: now also J1.17 (Pin_17)
- net KEY_IN_10: now also J1.19 (Pin_19)
- net KEY_IN_11: now also J1.21 (Pin_21)
- net KEY_IN_12: now also J1.23 (Pin_23)
- net KEY_IN_13: now also J1.25 (Pin_25)
- net KEY_IN_14: now also J1.27 (Pin_27)
- net KEY_IN_15: now also J1.29 (Pin_29)
- net KEY_IN_16: now also J1.31 (Pin_31)
- net KEY_IN_17: now also J1.33 (Pin_33)
- net KEY_IN_18: now also J1.35 (Pin_35)
- net KEY_IN_19: now also J2.1 (Pin_1)
- net KEY_IN_20: now also J2.3 (Pin_3)
- net KEY_IN_21: now also J2.5 (Pin_5)
- net KEY_IN_22: now also J2.7 (Pin_7)
- net KEY_IN_23: now also J2.9 (Pin_9)
- net KEY_IN_24: now also J2.11 (Pin_11)
- net KEY_IN_25: now also J2.13 (Pin_13)
- net KEY_IN_26: now also J2.15 (Pin_15)
- net KEY_IN_27: now also J2.17 (Pin_17)
- net KEY_IN_28: now also J2.19 (Pin_19)
- net KEY_IN_29: now also J2.21 (Pin_21)
- net KEY_IN_30: now also J2.23 (Pin_23)
- net KEY_IN_31: now also J2.25 (Pin_25)
- net KEY_IN_32: now also J2.27 (Pin_27)
- net KEY_IN_33: now also J2.29 (Pin_29)
- net KEY_IN_34: now also J2.31 (Pin_31)
- net KEY_IN_35: now also J2.33 (Pin_33)
- net KEY_IN_36: now also J2.35 (Pin_35)
- net KEY_OUT_01: now also J1.2 (Pin_2)
- net KEY_OUT_02: now also J1.4 (Pin_4)
- net KEY_OUT_03: now also J1.6 (Pin_6)
- net KEY_OUT_04: now also J1.8 (Pin_8)
- net KEY_OUT_05: now also J1.10 (Pin_10)
- net KEY_OUT_06: now also J1.12 (Pin_12)
- net KEY_OUT_07: now also J1.14 (Pin_14)
- net KEY_OUT_08: now also J1.16 (Pin_16)
- net KEY_OUT_09: now also J1.18 (Pin_18)
- net KEY_OUT_10: now also J1.20 (Pin_20)
- net KEY_OUT_11: now also J1.22 (Pin_22)
- net KEY_OUT_12: now also J1.24 (Pin_24)
- net KEY_OUT_13: now also J1.26 (Pin_26)
- net KEY_OUT_14: now also J1.28 (Pin_28)
- net KEY_OUT_15: now also J1.30 (Pin_30)
- net KEY_OUT_16: now also J1.32 (Pin_32)
- net KEY_OUT_17: now also J1.34 (Pin_34)
- net KEY_OUT_18: now also J1.36 (Pin_36)
- net KEY_OUT_19: now also J2.2 (Pin_2)
- net KEY_OUT_20: now also J2.4 (Pin_4)
- net KEY_OUT_21: now also J2.6 (Pin_6)
- net KEY_OUT_22: now also J2.8 (Pin_8)
- net KEY_OUT_23: now also J2.10 (Pin_10)
- net KEY_OUT_24: now also J2.12 (Pin_12)
- net KEY_OUT_25: now also J2.14 (Pin_14)
- net KEY_OUT_26: now also J2.16 (Pin_16)
- net KEY_OUT_27: now also J2.18 (Pin_18)
- net KEY_OUT_28: now also J2.20 (Pin_20)
- net KEY_OUT_29: now also J2.22 (Pin_22)
- net KEY_OUT_30: now also J2.24 (Pin_24)
- net KEY_OUT_31: now also J2.26 (Pin_26)
- net KEY_OUT_32: now also J2.28 (Pin_28)
- net KEY_OUT_33: now also J2.30 (Pin_30)
- net KEY_OUT_34: now also J2.32 (Pin_32)
- net KEY_OUT_35: now also J2.34 (Pin_34)
- net KEY_OUT_36: now also J2.36 (Pin_36)
- net VCC: now also J4.4 (Pin_4)
- no-connect marks 31 -> 39

Commit message: Cleanup of KiCAD area.
General cleanup. Added use of community libraries. Added schematics for encoder, rotor and programmer. Initial design review completed on schematics. Some initial PCB designs created (before schematic changes).
Parts:
- removed C13: GRM033Z71A104ME14D, SamacSys_Footprints:GRM033D70J224ME01D, symbol SamacSys_Parts:GRM033Z71A104ME14D
- removed C14: VJ0402A150FXQCW1BC, SamacSys_Footprints:CAPC1005X55N, symbol SamacSys_Parts:VJ0402A150FXQCW1BC
- removed IC1: EPM570T144C5N, SamacSys_Footprints:QFP50P2200X2200X160-144N, symbol SamacSys_Parts:EPM570T144C5N
- removed J3: Conn_02x06_Odd_Even, Connector_IDC:IDC-Header_2x06_P2.54mm_Vertical, symbol Connector_Generic:Conn_02x06_Odd_Even
- removed R1: ERJ-1GNF1001C, SamacSys_Footprints:ERJ1GN__0201_, symbol SamacSys_Parts:ERJ-1GNF1001C
- removed TP1, TP2, TP3, TP4: TestPoint_Small, TestPoint:TestPoint_Pad_D1.0mm, symbol Connector:TestPoint_Small
- removed Y1: SIT8918BAU71-33E-50.000000G, SamacSys_Footprints:SIT8918BAU7133E50000000G, symbol SamacSys_Parts:SIT8918BAU71-33E-50.000000G
- added C13, C14, C15, C16: GRM033Z71A104ME14D, Enigma_Components:GRM033D70J224ME01D, symbol Enigma_Conponents:GRM033Z71A104ME14D
- added IC1, IC2: EPM240T100C5N, Enigma_Components:QFP50P1600X1600X120-100N, symbol Enigma_Conponents:EPM240T100C5N
- added J3, J8: Conn_02x07_Odd_Even, Connector_IDC:IDC-Header_2x07_P2.54mm_Vertical, symbol Connector_Generic:Conn_02x07_Odd_Even
- added J5, J6: Conn_02x12_Odd_Even, Connector_IDC:IDC-Header_2x12_P2.54mm_Vertical, symbol Connector_Generic:Conn_02x12_Odd_Even
- added J7: Conn_02x01, Connector_PinHeader_2.54mm:PinHeader_2x01_P2.54mm_Vertical, symbol Connector_Generic:Conn_02x01
- added LED1, LED10, LED11, LED12, LED13, LED14, LED2, LED3, LED4, LED5, LED6, LED7, LED8, LED9: KT-0603R, Enigma_Components:LEDC1608X70N, symbol Enigma_Conponents:KT-0603R
- added R1, R10, R11, R12, R13, R14, R2, R3, R4, R5, R6, R7, R8, R9: ERA2AEB201X, Enigma_Components:ERA2AED122X, symbol Enigma_Conponents:ERA2AEB201X
- C1, C10, C11, C12, C2, C3, C4, C5, C6, C7, C8, C9: footprint SamacSys_Footprints:GRM033D70J224ME01D -> Enigma_Components:GRM033D70J224ME01D; symbol SamacSys_Parts:GRM033Z71A104ME14D -> Enigma_Conponents:GRM033Z71A104ME14D; Arrow Part Number (none) -> GRM033Z71A104ME14D; Arrow Price/Stock (none) -> https://www.arrow.com/en/products/grm033z71a104me14d/murata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; Description_1 (none) -> Multilayer Ceramic Capacitors MLCC - SMD/SMT .1UF 10V 20% 0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
Connections:
- net BIN_IN_01: now also IC1.1 (IO_1), J3.1 (Pin_1), J8.2 (Pin_2), R1.2
- net BIN_IN_02: now also IC1.2 (IO_2), J3.3 (Pin_3), J8.4 (Pin_4), R2.2
- net BIN_IN_03: now also IC1.3 (IO_3), J3.5 (Pin_5), J8.6 (Pin_6), R3.2
- net BIN_IN_04: now also IC1.4 (IO_4), J3.7 (Pin_7), J8.8 (Pin_8), R4.2
- net BIN_IN_05: now also IC1.5 (IO_5), J3.9 (Pin_9), J8.10 (Pin_10), R5.2
- net BIN_IN_06: now also IC1.6 (IO_6), J3.11 (Pin_11), J8.12 (Pin_12), R6.2
- net BIN_OUT_01: now also IC2.1 (IO_1), J3.2 (Pin_2), J8.1 (Pin_1), R8.2
- net BIN_OUT_02: now also IC2.2 (IO_2), J3.4 (Pin_4), J8.3 (Pin_3), R9.2
- net BIN_OUT_03: now also IC2.3 (IO_3), J3.6 (Pin_6), J8.5 (Pin_5), R10.2
- net BIN_OUT_04: now also IC2.4 (IO_4), J3.8 (Pin_8), J8.7 (Pin_7), R11.2
- net BIN_OUT_05: now also IC2.5 (IO_5), J3.10 (Pin_10), J8.9 (Pin_9), R12.2
- net BIN_OUT_06: now also IC2.6 (IO_6), J3.12 (Pin_12), J8.11 (Pin_11), R13.2
- net GND: now also C13.1, C14.1, C15.1, C16.1, IC1.10 (GNDIO_1), IC1.11 (GNDINT_1), IC1.32 (GNDIO_2), IC1.46 (GNDIO_3), IC1.60 (GNDIO_4), IC1.65 (GNDINT_2), IC1.79 (GNDIO_5), IC1.93 (GNDIO_6), IC2.10 (GNDIO_1), IC2.11 (GNDINT_1), IC2.32 (GNDIO_2), IC2.46 (GNDIO_3), IC2.60 (GNDIO_4), IC2.65 (GNDINT_2), IC2.79 (GNDIO_5), IC2.93 (GNDIO_6), J7.1 (Pin_1), LED1.1, LED10.1, LED11.1, LED12.1, LED13.1, LED2.1, LED3.1, LED4.1, LED5.1, LED6.1, LED8.1, LED9.1
- net JTAG_TCK: now also IC1.24 (TCK), IC2.24 (TCK)
- net JTAG_TDI: now also IC1.23 (TDI)
- net JTAG_TDO: now also IC2.25 (TDO)
- net JTAG_TMS: now also IC1.22 (TMS), IC2.22 (TMS)
- net KEY_IN_01: now also IC2.26 (IO_16), J5.2 (Pin_2); no longer J1.1 (Pin_1)
- net KEY_IN_02: now also IC2.27 (IO_17), J5.4 (Pin_4); no longer J1.3 (Pin_3)
- net KEY_IN_03: now also IC2.28 (IO_18), J5.6 (Pin_6); no longer J1.5 (Pin_5)
- net KEY_IN_04: now also IC2.29 (IO_19), J5.8 (Pin_8); no longer J1.7 (Pin_7)
- net KEY_IN_05: now also IC2.30 (IO_20), J5.10 (Pin_10); no longer J1.9 (Pin_9)
- net KEY_IN_06: now also IC2.33 (IO_21), J5.12 (Pin_12); no longer J1.11 (Pin_11)
- net KEY_IN_07: now also IC2.34 (IO_22), J5.14 (Pin_14); no longer J1.13 (Pin_13)
- net KEY_IN_08: now also IC2.35 (IO_23), J5.16 (Pin_16); no longer J1.15 (Pin_15)
- net KEY_IN_09: now also IC2.36 (IO_24), J5.18 (Pin_18); no longer J1.17 (Pin_17)
- net KEY_IN_10: now also IC2.37 (IO_25), J5.20 (Pin_20); no longer J1.19 (Pin_19)
- net KEY_IN_11: now also IC2.38 (IO_26), J5.22 (Pin_22); no longer J1.21 (Pin_21)
- net KEY_IN_12: now also IC2.39 (IO_27), J5.24 (Pin_24); no longer J1.23 (Pin_23)
- net KEY_IN_13: now also J1.2 (Pin_2), IC2.40 (IO_28); no longer J1.25 (Pin_25)
- net KEY_IN_14: now also J1.4 (Pin_4), IC2.41 (IO_29); no longer J1.27 (Pin_27)
- net KEY_IN_15: now also J1.6 (Pin_6), IC2.42 (IO_30); no longer J1.29 (Pin_29)
- net KEY_IN_16: now also J1.8 (Pin_8), IC2.47 (IO_31); no longer J1.31 (Pin_31)
- net KEY_IN_17: now also J1.10 (Pin_10), IC2.48 (IO_32); no longer J1.33 (Pin_33)
- net KEY_IN_18: now also J1.12 (Pin_12), IC2.49 (IO_33); no longer J1.35 (Pin_35)
- net KEY_IN_19: now also J1.14 (Pin_14), IC2.50 (IO_34); no longer J2.1 (Pin_1)
- net KEY_IN_20: now also J1.16 (Pin_16), IC2.51 (IO_35); no longer J2.3 (Pin_3)
- net KEY_IN_21: now also J1.18 (Pin_18), IC2.52 (IO_36); no longer J2.5 (Pin_5)
- net KEY_IN_22: now also J1.20 (Pin_20), IC2.53 (IO_37); no longer J2.7 (Pin_7)
- net KEY_IN_23: now also J1.22 (Pin_22), IC2.54 (IO_38); no longer J2.9 (Pin_9)
- net KEY_IN_24: now also J1.24 (Pin_24), IC2.55 (IO_39); no longer J2.11 (Pin_11)
- net KEY_IN_25: now also J1.26 (Pin_26), IC2.56 (IO_40); no longer J2.13 (Pin_13)
- net KEY_IN_26: now also J1.28 (Pin_28), IC2.57 (IO_41); no longer J2.15 (Pin_15)
- net KEY_IN_27: now also J1.30 (Pin_30), IC2.58 (IO_42); no longer J2.17 (Pin_17)
- net KEY_IN_28: now also J1.32 (Pin_32), IC2.66 (IO_44); no longer J2.19 (Pin_19)
- net KEY_IN_29: now also J1.34 (Pin_34), IC2.67 (IO_45); no longer J2.21 (Pin_21)
- net KEY_IN_30: now also J1.36 (Pin_36), IC2.68 (IO_46); no longer J2.23 (Pin_23)
- net KEY_IN_31: now also J1.38 (Pin_38), IC2.69 (IO_47); no longer J2.25 (Pin_25)
- net KEY_IN_32: now also J1.40 (Pin_40), IC2.70 (IO_48); no longer J2.27 (Pin_27)
- net KEY_IN_33: now also J2.2 (Pin_2), IC2.71 (IO_49); no longer J2.29 (Pin_29)
- net KEY_IN_34: now also J2.4 (Pin_4), IC2.72 (IO_50); no longer J2.31 (Pin_31)
- net KEY_IN_35: now also J2.6 (Pin_6), IC2.73 (IO_51); no longer J2.33 (Pin_33)
- net KEY_IN_36: now also J2.8 (Pin_8), IC2.74 (IO_52); no longer J2.35 (Pin_35)
- net KEY_OUT_01: now also IC1.26 (IO_16), J5.1 (Pin_1); no longer J1.2 (Pin_2)
- net KEY_OUT_02: now also IC1.27 (IO_17), J5.3 (Pin_3); no longer J1.4 (Pin_4)
- net KEY_OUT_03: now also IC1.28 (IO_18), J5.5 (Pin_5); no longer J1.6 (Pin_6)
- net KEY_OUT_04: now also IC1.29 (IO_19), J5.7 (Pin_7); no longer J1.8 (Pin_8)
- net KEY_OUT_05: now also IC1.30 (IO_20), J5.9 (Pin_9); no longer J1.10 (Pin_10)
- net KEY_OUT_06: now also IC1.33 (IO_21), J5.11 (Pin_11); no longer J1.12 (Pin_12)
- net KEY_OUT_07: now also IC1.34 (IO_22), J5.13 (Pin_13); no longer J1.14 (Pin_14)
- net KEY_OUT_08: now also IC1.35 (IO_23), J5.15 (Pin_15); no longer J1.16 (Pin_16)
- net KEY_OUT_09: now also IC1.36 (IO_24), J5.17 (Pin_17); no longer J1.18 (Pin_18)
- net KEY_OUT_10: now also IC1.37 (IO_25), J5.19 (Pin_19); no longer J1.20 (Pin_20)
- net KEY_OUT_11: now also IC1.38 (IO_26), J5.21 (Pin_21); no longer J1.22 (Pin_22)
- net KEY_OUT_12: now also IC1.39 (IO_27), J5.23 (Pin_23); no longer J1.24 (Pin_24)
- net KEY_OUT_13: now also J1.1 (Pin_1), IC1.40 (IO_28); no longer J1.26 (Pin_26)
- net KEY_OUT_14: now also J1.3 (Pin_3), IC1.41 (IO_29); no longer J1.28 (Pin_28)
- net KEY_OUT_15: now also J1.5 (Pin_5), IC1.42 (IO_30); no longer J1.30 (Pin_30)
- net KEY_OUT_16: now also J1.7 (Pin_7), IC1.47 (IO_31); no longer J1.32 (Pin_32)
- net KEY_OUT_17: now also J1.9 (Pin_9), IC1.48 (IO_32); no longer J1.34 (Pin_34)
- net KEY_OUT_18: now also J1.11 (Pin_11), IC1.49 (IO_33); no longer J1.36 (Pin_36)
- net KEY_OUT_19: now also J1.13 (Pin_13), IC1.50 (IO_34); no longer J2.2 (Pin_2)
- net KEY_OUT_20: now also J1.15 (Pin_15), IC1.51 (IO_35); no longer J2.4 (Pin_4)
- net KEY_OUT_21: now also J1.17 (Pin_17), IC1.52 (IO_36); no longer J2.6 (Pin_6)
- net KEY_OUT_22: now also J1.19 (Pin_19), IC1.53 (IO_37); no longer J2.8 (Pin_8)
- net KEY_OUT_23: now also J1.21 (Pin_21), IC1.54 (IO_38); no longer J2.10 (Pin_10)
- net KEY_OUT_24: now also J1.23 (Pin_23), IC1.55 (IO_39); no longer J2.12 (Pin_12)
- net KEY_OUT_25: now also J1.25 (Pin_25), IC1.56 (IO_40); no longer J2.14 (Pin_14)
- net KEY_OUT_26: now also J1.27 (Pin_27), IC1.57 (IO_41); no longer J2.16 (Pin_16)
- net KEY_OUT_27: now also J1.29 (Pin_29), IC1.58 (IO_42); no longer J2.18 (Pin_18)
- net KEY_OUT_28: now also J1.31 (Pin_31), IC1.66 (IO_44); no longer J2.20 (Pin_20)
- net KEY_OUT_29: now also J1.33 (Pin_33), IC1.67 (IO_45); no longer J2.22 (Pin_22)
- net KEY_OUT_30: now also J1.35 (Pin_35), IC1.68 (IO_46); no longer J2.24 (Pin_24)
- net KEY_OUT_31: now also J1.37 (Pin_37), IC1.69 (IO_47); no longer J2.26 (Pin_26)
- net KEY_OUT_32: now also J1.39 (Pin_39), IC1.70 (IO_48); no longer J2.28 (Pin_28)
- net KEY_OUT_33: now also J2.1 (Pin_1), IC1.71 (IO_49); no longer J2.30 (Pin_30)
- net KEY_OUT_34: now also J2.3 (Pin_3), IC1.72 (IO_50); no longer J2.32 (Pin_32)
- net KEY_OUT_35: now also J2.5 (Pin_5), IC1.73 (IO_51); no longer J2.34 (Pin_34)
- net KEY_OUT_36: now also J2.7 (Pin_7), IC1.74 (IO_52); no longer J2.36 (Pin_36)
- net VCC: now also C13.2, C14.2, C15.2, C16.2, IC1.13 (VCCINT_1), IC1.31 (VCCIO1_2), IC1.45 (VCCIO1_3), IC1.59 (VCCIO2_1), IC1.63 (VCCINT_2), IC1.80 (VCCIO2_2), IC1.9 (VCCIO1_1), IC1.94 (VCCIO2_3), IC2.13 (VCCINT_1), IC2.31 (VCCIO1_2), IC2.45 (VCCIO1_3), IC2.59 (VCCIO2_1), IC2.63 (VCCINT_2), IC2.80 (VCCIO2_2), IC2.9 (VCCIO1_1), IC2.94 (VCCIO2_3), J7.2 (Pin_2), R14.2, R7.2
- net KEY_OUT_51: now reaches J2.37 (Pin_37)
- net KEY_OUT_51: now also IC1.91 (IO_67)
- net KEY_IN_51: now reaches J2.38 (Pin_38)
- net KEY_IN_51: now also IC2.91 (IO_67)
- net KEY_OUT_52: now reaches J2.39 (Pin_39)
- net KEY_OUT_52: now also IC1.92 (IO_68)
- net KEY_IN_52: now reaches J2.40 (Pin_40)
- net KEY_IN_52: now also IC2.92 (IO_68)
- new net: LED5.2, R5.1
- new net: LED13.2, R13.1
- new net: LED12.2, R12.1
- new net: LED1.2, R1.1
- new net: LED8.2, R8.1
- new net: LED4.2, R4.1
- new net: LED3.2, R3.1
- new net: LED7.2, R7.1
- new net: LED11.2, R11.1
- new net: LED10.2, R10.1
- new net: LED14.2, R14.1
- new net: LED9.2, R9.1
- new net: LED2.2, R2.1
- new net: LED6.2, R6.1
- new net BIN_IN_EN: IC1.7 (IO_7), J3.13 (Pin_13), J8.14 (Pin_14), LED7.1
- new net BIN_OUT_EN: IC2.7 (IO_7), J3.14 (Pin_14), J8.13 (Pin_13), LED14.1
- new net JTAG_TDX: IC1.25 (TDO), IC2.23 (TDI)
- new net KEY_IN_37: IC2.75 (IO_53), J2.10 (Pin_10)
- new net KEY_IN_38: IC2.76 (IO_54), J2.12 (Pin_12)
- new net KEY_IN_39: IC2.77 (IO_55), J2.14 (Pin_14)
- new net KEY_IN_40: IC2.78 (IO_56), J2.16 (Pin_16)
- new net KEY_IN_41: IC2.81 (IO_57), J2.18 (Pin_18)
- new net KEY_IN_42: IC2.82 (IO_58), J2.20 (Pin_20)
- new net KEY_IN_43: IC2.83 (IO_59), J2.22 (Pin_22)
- new net KEY_IN_44: IC2.84 (IO_60), J2.24 (Pin_24)
- new net KEY_IN_45: IC2.85 (IO_61), J2.26 (Pin_26)
- new net KEY_IN_46: IC2.86 (IO_62), J2.28 (Pin_28)
- new net KEY_IN_47: IC2.87 (IO_63), J2.30 (Pin_30)
- new net KEY_IN_48: IC2.88 (IO_64), J2.32 (Pin_32)
- new net KEY_IN_49: IC2.89 (IO_65), J2.34 (Pin_34)
- new net KEY_IN_50: IC2.90 (IO_66), J2.36 (Pin_36)
- new net KEY_IN_53: IC2.95 (IO_69), J6.2 (Pin_2)
- new net KEY_IN_54: IC2.96 (IO_70), J6.4 (Pin_4)
- new net KEY_IN_55: IC2.97 (IO_71), J6.6 (Pin_6)
- new net KEY_IN_56: IC2.98 (IO_72), J6.8 (Pin_8)
- new net KEY_IN_57: IC2.99 (IO_73), J6.10 (Pin_10)
- new net KEY_IN_58: IC2.100 (IO_74), J6.12 (Pin_12)
- new net KEY_IN_59: IC2.15 (IO_9), J6.14 (Pin_14)
- new net KEY_IN_60: IC2.16 (IO_10), J6.16 (Pin_16)
- new net KEY_IN_61: IC2.17 (IO_11), J6.18 (Pin_18)
- new net KEY_IN_62: IC2.18 (IO_12), J6.20 (Pin_20)
- new net KEY_IN_63: IC2.19 (IO_13), J6.22 (Pin_22)
- new net KEY_IN_64: IC2.20 (IO_14), J6.24 (Pin_24)
- new net KEY_OUT_37: IC1.75 (IO_53), J2.9 (Pin_9)
- new net KEY_OUT_38: IC1.76 (IO_54), J2.11 (Pin_11)
- new net KEY_OUT_39: IC1.77 (IO_55), J2.13 (Pin_13)
- new net KEY_OUT_40: IC1.78 (IO_56), J2.15 (Pin_15)
- new net KEY_OUT_41: IC1.81 (IO_57), J2.17 (Pin_17)
- new net KEY_OUT_42: IC1.82 (IO_58), J2.19 (Pin_19)
- new net KEY_OUT_43: IC1.83 (IO_59), J2.21 (Pin_21)
- new net KEY_OUT_44: IC1.84 (IO_60), J2.23 (Pin_23)
- new net KEY_OUT_45: IC1.85 (IO_61), J2.25 (Pin_25)
- new net KEY_OUT_46: IC1.86 (IO_62), J2.27 (Pin_27)
- new net KEY_OUT_47: IC1.87 (IO_63), J2.29 (Pin_29)
- new net KEY_OUT_48: IC1.88 (IO_64), J2.31 (Pin_31)
- new net KEY_OUT_49: IC1.89 (IO_65), J2.33 (Pin_33)
- new net KEY_OUT_50: IC1.90 (IO_66), J2.35 (Pin_35)
- new net KEY_OUT_53: IC1.95 (IO_69), J6.1 (Pin_1)
- new net KEY_OUT_54: IC1.96 (IO_70), J6.3 (Pin_3)
- new net KEY_OUT_55: IC1.97 (IO_71), J6.5 (Pin_5)
- new net KEY_OUT_56: IC1.98 (IO_72), J6.7 (Pin_7)
- new net KEY_OUT_57: IC1.99 (IO_73), J6.9 (Pin_9)
- new net KEY_OUT_58: IC1.100 (IO_74), J6.11 (Pin_11)
- new net KEY_OUT_59: IC1.15 (IO_9), J6.13 (Pin_13)
- new net KEY_OUT_60: IC1.16 (IO_10), J6.15 (Pin_15)
- new net KEY_OUT_61: IC1.17 (IO_11), J6.17 (Pin_17)
- new net KEY_OUT_62: IC1.18 (IO_12), J6.19 (Pin_19)
- new net KEY_OUT_63: IC1.19 (IO_13), J6.21 (Pin_21)
- new net KEY_OUT_64: IC1.20 (IO_14), J6.23 (Pin_23)
- no-connect marks 39 -> 21
Other:
- note added: "- reflector -"
- note added: "- stator -"
- note added: "--------------- Pin Mappings (Stator) -------------------- KEY_IN_xx => BIN_OUT_0x : Input from Keyboard, Output to Rotor [SND] BIN_IN_0x => KEY_OUT_xx : Input from Rotor [RTN], Output to Lightboard --------------- Pin Mappings (Reflector) ----------------- BIN_IN_0x => KEY_OUT_xx : Input from Rotor [SND], Output to Plugboard KEY_IN_xx => BIN_OUT_0x : Input from Plugboard, Output to Rotor [RTN]"
- note added: "Decoder"
- note added: "Encoder"
- note added: "Programming Interface"
- note added: "Reflector Interface"
- note removed: "-------------------- Pin Mappings -------------------- BIN_IN_0x => KEY_OUT_xx : Input from Rotor [SND], Output to Plugboard KEY_IN_xx => BIN_OUT_0x : Input from Plugboard, Output to Rotor [RTN]"
- company: (none) -> Enigmatic
- title: Enigma Stator/Reflector Controller -> Enigma - Stator/Reflector
- moved on the sheet: C1, C10, C11, C12, C2, C3, C4, C5, C6, C7, C8, C9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
