File: Electronics/KiCad/enigma_debugger/enigma_debugger.kicad_pcb (KiCad board)
At the start: 4 copper layers, 82.2 x 56.5 mm, 59 parts, among them J1 Conn_02x07_Odd_Even, J2 Conn_02x07_Odd_Even, J3 Conn_01x02

Commit message: Production fab updates.
Routing:
- net Net-(J1-Pin_14): track 104.3 -> 103.6 mm, vias 0 -> 1
